Commit message: fix mesh folder path to spawn robot correctly

File: Assets/URDF/scout_v2.urdf (robot description, URDF)
Before this commit: robot scout_v2, 6 links, 5 joints
Links:
- link base_link: geometry collision box size=0.15416666666666667 0.627 0.06999999999999999; collision box size=0.925 0.38 0.21
- link front_left_wheel_link: geometry collision cylinder length=0.11653 radius=0.16459; visual mesh filename=package://scout/scout_description/meshes/wheel_type1.dae
- link front_right_wheel_link: geometry collision cylinder length=0.11653 radius=0.16459; visual mesh filename=package://scout/scout_description/meshes/wheel_type1.dae
- link rear_left_wheel_link: geometry collision cylinder length=0.11653 radius=0.16459; visual mesh filename=package://scout/scout_description/meshes/wheel_type1.dae
- link rear_right_wheel_link: geometry collision cylinder length=0.11653 radius=0.16459; visual mesh filename=package://scout/scout_description/meshes/wheel_type1.dae
