Commit message: include laser and camera  in scout  urdf include  sensor meshs path include scripts for laser plugin (not fineshed yet)

File: Assets/URDF/scout/scout_description/urdf/scout_v2.urdf (robot description, URDF)
Before this commit: robot scout_v2, 6 links, 5 joints
Links:
- added link centercolor
- added link centerdepth
- added link centerired1
- added link centerired2
- added link centerrs200_camera
Joints:
- added joint centercolor_joint: type fixed, parent centerrs200_camera, child centercolor, origin xyz=0 -0.046 0.004 rpy=1.5707963267948966 3.141592653589793 1.5707963267948966
- added joint centerdepth_joint: type fixed, parent centerrs200_camera, child centerdepth, origin xyz=0 -0.03 0.004 rpy=0 0 0
- added joint centerired1_joint: type fixed, parent centerrs200_camera, child centerired1, origin xyz=0 -0.06 0.004 rpy=0 0 0
- added joint centerired2_joint: type fixed, parent centerrs200_camera, child centerired2, origin xyz=0 0.01 0.004 rpy=0 0 0
- added joint centerrealsense_joint: type fixed, parent base_link, child centerrs200_camera, origin xyz=0.0695 0 0.662 rpy=0 0 0

File: Assets/URDF/scout/scout_description/urdf/scout_v2.xacro (robot description, xacro)
@@ -6,4 +6,6 @@
     <xacro:include filename="$(find scout_description)/urdf/scout_wheel_type1.xacro" />
     <xacro:include filename="$(find scout_description)/urdf/scout_wheel_type2.xacro" />
+    <!-- ### Realsense camera include ###-->
+    <xacro:include filename="$(find scout_description)/urdf/realsense-RS200.macro.xacro"/>
     <!-- Variables -->
     <xacro:property name="M_PI" value="3.14159"/>
@@ -17,4 +19,8 @@
     <xacro:property name="wheel_length" value="1.1653e-01" />
     <xacro:property name="wheel_radius" value="1.6459e-01" />
+    <!-- center -->
+    <xacro:realsense-rs200 prefix="center" parent="base_link">
+        <origin xyz="0.0695 0 0.662" rpy="0 0 0" />
+    </xacro:realsense-rs200>
     <!-- Base link -->
     <link name="base_link">

File: Assets/URDF/scout_v2.urdf (robot description, URDF)
Before this commit: robot scout_v2, 6 links, 5 joints
Links:
- added link base_camera_link, mass 0.001
- added link base_camera_optical_frame, mass 0.001
- added link laser_link, mass 0.00833634573995571; collision mesh filename=package://sensors/meshes/laser_link_collision.STL; visual mesh filename=package://sensors/meshes/laser_link.STL
Joints:
- added joint base_camera_joint: type fixed, parent base_link, child base_camera_link, origin xyz=0.3895 0 0.094 rpy=0 0 0
- added joint base_camera_optical_joint: type fixed, parent base_camera_link, child base_camera_optical_frame, origin xyz=0 0 0 rpy=1.5707963267966 0 1.5707963267966
- added joint laser_joint: type fixed, parent base_link, child laser_link, origin xyz=0.235 0 0.23 rpy=0 0 3.14, axis 0 0 0
